File: PCB/FT817_buddy_v4/FT817_buddy_v4.sch (KiCad schematic (older format))
At the start: 65 parts, among them J1 FT817_ACC, J2 KEY_OUT, J3 KEY_IN, J4 K16 CW processor, J5 GND, J6 EXP PWR SELECT, J7 , J8 , J9 EXPANSION HEADER, SW1 SW_Push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

Commit message: Updated with input/ouput and not connected symbols
Connections:
- no-connect marks 0 -> 18
Other:
- note added: "20 March 2021"
- note removed: "5 December 2020"
Changed lines of the file:
@@
 	-1   0    0    1
 $EndComp
-Text GLabel 1050 4250 3    50   Input ~ 0
+Text GLabel 1050 4250 3    50   UnSpc ~ 0
 GND1
 Text GLabel 1150 4250 3    50   Input ~ 0
 VDD1
-Text GLabel 1250 4250 3    50   Input ~ 0
-GND2
-Text GLabel 1350 4250 3    50   Input ~ 0
+Text GLabel 1250 4250 3    50   UnSpc ~ 0
+GND2
+Text GLabel 1350 4250 3    50   Output ~ 0
 VDD2
-Text GLabel 1250 2850 0    50   Input ~ 0
+Text GLabel 1250 2850 0    50   UnSpc ~ 0
 GND1
-Text GLabel 2250 2850 2    50   Input ~ 0
+Text GLabel 2250 2850 2    50   UnSpc ~ 0
 GND2
 Text GLabel 1050 2450 0    50   Input ~ 0
@@
 Text GLabel 2450 2450 2    50   Input ~ 0
 VDD2
-Text GLabel 5950 1000 2    50   Input ~ 0
+Text GLabel 5950 1000 2    50   Output ~ 0
 VDD1
-Text GLabel 4850 1400 3    50   Input ~ 0
+Text GLabel 4850 1500 3    50   UnSpc ~ 0
 GND1
-Text GLabel 1150 1100 2    50   Input ~ 0
+Text GLabel 1150 1100 2    50   UnSpc ~ 0
 GND1
-Text GLabel 1150 1000 2    50   Input ~ 0
+Text GLabel 1150 1000 2    50   Output ~ 0
 FT817_Vout
 Text GLabel 2900 1000 0    50   Input ~ 0
@@
 Text GLabel 1150 1400 2    50   Input ~ 0
 FT817_RXD
-Text GLabel 1150 1300 2    50   Input ~ 0
+Text GLabel 1150 1300 2    50   Output ~ 0
 FT817_TXD
-Text GLabel 1150 1200 2    50   Input ~ 0
+Text GLabel 1150 1200 2    50   UnSpc ~ 0
 SHIELD
 Text GLabel 1250 2750 0    50   Input ~ 0
 FT817_TXD
-Text GLabel 1250 2550 0    50   Input ~ 0
+Text GLabel 1250 2550 0    50   Output ~ 0
 FT817_RXD
 Text GLabel 3850 4100 1    50   Input ~ 0
 VDD2
-Text GLabel 3750 6100 3    50   Input ~ 0
-GND2
-Text GLabel 2250 2750 2    50   Input ~ 0
+Text GLabel 3750 6100 3    50   UnSpc ~ 0
+GND2
+Text GLabel 2250 2750 2    50   Output ~ 0
 ARD_RXD
 Text GLabel 2250 2550 2    50   Input ~ 0
 ARD_TXD
-Text GLabel 2250 4400 0    50   Input ~ 0
+Text GLabel 2250 4400 0    50   Output ~ 0
 ARD_TXD
-Text GLabel 3150 5300 0    50   Input ~ 0
+Text GLabel 3150 5300 0    50   Output ~ 0
 BACKLIGHT
-Text GLabel 9250 3000 0    50   Input ~ 0
+Text GLabel 9250 3000 0    50   UnSpc ~ 0
 GND2
 Text GLabel 8750 4150 0    50   Input ~ 0
@@
 Text GLabel 8350 3350 0    50   Input ~ 0
 RST
-Text GLabel 3150 5200 0    50   Input ~ 0
+Text GLabel 3150 5200 0    50   Output ~ 0
 CLK
-Text GLabel 3150 5100 0    50   Input ~ 0
+Text GLabel 3150 5100 0    50   Output ~ 0
 DIN
-Text GLabel 3150 5000 0    50   Input ~ 0
+Text GLabel 3150 5000 0    50   Output ~ 0
 DC
-Text GLabel 3150 4900 0    50   Input ~ 0
+Text GLabel 3150 4900 0    50   Output ~ 0
 CE
-Text GLabel 3150 4800 0    50   Input ~ 0
+Text GLabel 3150 4800 0    50   Output ~ 0
 RST
-Text GLabel 3150 5500 0    50   Input ~ 0
+Text GLabel 1300 7050 0    50   UnSpc ~ 0
+GND2
+Text GLabel 2350 7050 0    50   UnSpc ~ 0
+GND2
+Text GLabel 3400 7050 0    50   UnSpc ~ 0
+GND2
+Text GLabel 1700 7050 2    50   Output ~ 0
+SW7
+Text GLabel 2750 7050 2    50   Output ~ 0
 SW8
-Text GLabel 3150 5400 0    50   Input ~ 0
-SW9
-Text GLabel 1300 7050 0    50   Input ~ 0
-GND2
-Text GLabel 2350 7050 0    50   Input ~ 0
-GND2
-Text GLabel 3400 7050 0    50   Input ~ 0
-GND2
-Text GLabel 1700 7050 2    50   Input ~ 0
-SW7
-Text GLabel 2750 7050 2    50   Input ~ 0
-SW8
-Text GLabel 3800 7050 2    50   Input ~ 0
+Text GLabel 3800 7050 2    50   Output ~ 0
 SW9
 $Comp
@@
 	1    0    0    -1
 $EndComp
-Text GLabel 1150 2050 1    50   Input ~ 0
+Text GLabel 1150 2050 1    50   UnSpc ~ 0
 GND1
-Text GLabel 2350 2050 1    50   Input ~ 0
+Text GLabel 2350 2050 1    50   UnSpc ~ 0
 GND2
 Wire Wire Line
@@
 Wire Wire Line
 	9450 4050 9800 4050
-Text GLabel 3750 4100 1    50   Input ~ 0
+Text GLabel 3750 4100 1    50   Output ~ 0
 3V3
 Wire Wire Line
@@
 	-1   0    0    1
 $EndComp
-Text GLabel 3150 5600 0    50   Input ~ 0
-SW7
 Text GLabel 2250 4250 0    50   Input ~ 0
 ARD_RXD
@@
 	1    0    0    -1
 $EndComp
-Text GLabel 3350 3150 0    50   Input ~ 0
+Text GLabel 3350 3150 0    50   Output ~ 0
 KEY
-Text GLabel 3350 3250 0    50   Input ~ 0
+Text GLabel 3350 3250 0    50   Output ~ 0
 SIDETONE
 Text GLabel 3350 3350 0    50   Input ~ 0
@@
 Text GLabel 4350 3150 2    50   Input ~ 0
 LEFT_PADDLE
-Text GLabel 4350 3050 2    50   Input ~ 0
+Text GLabel 4350 3050 2    50   UnSpc ~ 0
 GND2
 Text GLabel 3350 3050 0    50   Input ~ 0
@@
 Wire Wire Line
 	3650 3350 3350 3350
-Text GLabel 8500 1550 2    50   Input ~ 0
+Text GLabel 8500 1550 2    50   Output ~ 0
 LEFT_PADDLE
-Text GLabel 8500 1250 2    50   Input ~ 0
+Text GLabel 8500 1250 2    50   Output ~ 0
 RIGHT_PADDLE
-Text GLabel 8500 850  2    50   Input ~ 0
+Text GLabel 8500 850  2    50   UnSpc ~ 0
 GND2
 $Comp
@@
 	1    0    0    -1
 $EndComp
-Text GLabel 7450 4400 0    50   Input ~ 0
+Text GLabel 7300 4400 0    50   UnSpc ~ 0
 GND2
 Wire Wire Line
@@
 Wire Wire Line
 	1800 5100 1800 5150
-Text GLabel 1200 5950 0    50   Input ~ 0
+Text GLabel 1200 5950 0    50   UnSpc ~ 0
 GND2
 Wire Wire Line
 	1800 5850 1800 5950
-Text GLabel 10450 1150 2    50   Input ~ 0
+Text GLabel 10550 1150 2    50   UnSpc ~ 0
 GND2
 Wire Wire Line
 	4150 5100 5100 5100
-Text GLabel 4150 5200 2    50   Input ~ 0
+Text GLabel 4150 5200 2    50   Output ~ 0
 KEY_SW1
-Text GLabel 4150 5300 2    50   Input ~ 0
+Text GLabel 4150 5300 2    50   Output ~ 0
 KEY_SW2
-Text GLabel 4150 5400 2    50   Input ~ 0
+Text GLabel 4150 5400 2    50   Output ~ 0
 KEY_SW3
-Text GLabel 3150 5800 0    50   Input ~ 0
+Text GLabel 3150 5800 0    50   Output ~ 0
 KEY_SW4
 Text GLabel 5750 2950 0    50   Input ~ 0
@@
 Text GLabel 5750 3250 0    50   Input ~ 0
 KEY_SW4
-Text GLabel 6150 3850 3    50   Input ~ 0
-GND2
-Text GLabel 7350 2050 0    50   Input ~ 0
+Text GLabel 6150 3850 3    50   UnSpc ~ 0
+GND2
+Text GLabel 7350 2050 0    50   Output ~ 0
 PBNET
 Wire Wire Line
@@
 Text GLabel 5750 3350 0    50   Input ~ 0
 KEY
-Text GLabel 6550 3350 2    50   Input ~ 0
+Text GLabel 6550 3350 2    50   Output ~ 0
 KEY_OUT
 Text GLabel 10350 1550 2    50   Input ~ 0
@@
 Text GLabel 5750 3450 0    50   Input ~ 0
 BACKLIGHT
-Text GLabel 6550 3450 2    50   Input ~ 0
+Text GLabel 6550 3450 2    50   Output ~ 0
 LIGHT_OUT
 Text GLabel 9900 6200 2    50   Input ~ 0
@@
 	0    -1   -1   0
 $EndComp
-Text GLabel 7950 2550 2    50   Input ~ 0
+Text GLabel 7950 2550 2    50   UnSpc ~ 0
 GND2
 Wire Wire Line
@@
 	-1   0    0    1
 $EndComp
-Text GLabel 1150 800  2    50   Input ~ 0
+Text GLabel 1150 800  2    50   UnSpc ~ 0
 GND1
-Text GLabel 5900 5100 2    50   Input ~ 0
-GND2
-Text GLabel 5900 5550 2    50   Input ~ 0
-GND2
-Text GLabel 5900 6000 2    50   Input ~ 0
+Text GLabel 5900 5100 2    50   UnSpc ~ 0
+GND2
+Text GLabel 5900 5550 2    50   UnSpc ~ 0
+GND2
+Text GLabel 5900 6000 2    50   UnSpc ~ 0
 GND2
 Connection ~ 5100 6900
@@
 	-1   0    0    -1
 $EndComp
-Text GLabel 5900 7350 2    50   Input ~ 0
-GND2
-Text GLabel 5900 6900 2    50   Input ~ 0
-GND2
-Text GLabel 5900 6450 2    50   Input ~ 0
+Text GLabel 5900 7350 2    50   UnSpc ~ 0
+GND2
+Text GLabel 5900 6900 2    50   UnSpc ~ 0
+GND2
+Text GLabel 5900 6450 2    50   UnSpc ~ 0
 GND2
 Text Notes 7200 7050 0    50   ~ 0
@@
 FT-817 Buddy Schematic Rev4
 Text Notes 8150 7650 0    50   ~ 0
-5 December 2020
+20 March 2021
 Text Notes 10600 7650 0    50   ~ 0
 4
@@
 Wire Wire Line
 	6900 5250 7350 5250
-Text GLabel 7350 5150 0    50   Input ~ 0
-GND2
-Text GLabel 4150 5500 2    50   Input ~ 0
+Text GLabel 7350 5150 0    50   UnSpc ~ 0
+GND2
+Text GLabel 4150 5500 2    50   BiDi ~ 0
 EXP_SDA
-Text GLabel 4150 5600 2    50   Input ~ 0
+Text GLabel 4150 5600 2    50   Output ~ 0
 EXP_SCL
-Text GLabel 7350 4850 0    50   Input ~ 0
+Text GLabel 7350 4850 0    50   BiDi ~ 0
 EXP_SDA
 Text GLabel 7350 4950 0    50   Input ~ 0
 EXP_SCL
-Text GLabel 7350 5050 0    50   Input ~ 0
+Text GLabel 7350 5050 0    50   Output ~ 0
 EXP_SQW
 Text GLabel 3150 4700 0    50   Input ~ 0
@@
 Text Notes 7200 6800 0    118  ~ 0
 FT-817 Buddy
+NoConn ~ 4150 3350
+NoConn ~ 3150 5700
+NoConn ~ 4150 5800
+NoConn ~ 4150 5700
+NoConn ~ 4150 4900
+NoConn ~ 4150 4600
+NoConn ~ 4150 4500
+NoConn ~ 3550 4100
+NoConn ~ 3650 6100
+NoConn ~ 10350 1350
+NoConn ~ 10350 1450
+NoConn ~ 7900 1350
+NoConn ~ 7900 1450
+NoConn ~ 6550 2850
+NoConn ~ 5750 3550
+NoConn ~ 5750 3650
+NoConn ~ 6550 3650
+NoConn ~ 6550 3550
+Text GLabel 3150 5600 0    50   Input ~ 0
+SW7
+Text GLabel 3150 5500 0    50   Input ~ 0
+SW8
+Text GLabel 3150 5400 0    50   Input ~ 0
+SW9
+Wire Wire Line
+	10450 1150 10550 1150
+Connection ~ 10450 1150
+Wire Wire Line
+	7300 4400 7450 4400
+Wire Wire Line
+	4850 1400 4850 1500
 $EndSCHEMATC
